File: PCB/ChuniController/IRBlaster.kicad_sch (KiCad schematic)
At the start: 5 parts, among them Q7 AO3400

Commit message: PCB
Connections:
- net 3V3 renamed 5V
Changed lines of the file:
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@@
 		)
 	)
-	(hierarchical_label "3V3"
+	(hierarchical_label "5V"
 		(shape input)
 		(at 50.8 66.04 180)

Commit message: PCB Add pullup 10kR in LM393D reduce AO3400 pulldown to 10kR
Parts:
- R11: value 100K -> 10K
Other:
- moved on the sheet: R11
Changed lines of the file:
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@@
 	(wire
 		(pts
-			(xy 68.58 71.12) (xy 68.58 76.2)
+			(xy 68.58 71.12) (xy 68.58 74.93)
 		)
 		(stroke
@@
 		(pts
 			(xy 50.8 83.82) (xy 68.58 83.82)
+		)
+		(stroke
+			(width 0)
+			(type default)
+		)
+	)
+	(wire
+		(pts
+			(xy 68.58 82.55) (xy 68.58 83.82)
 		)
 		(stroke
@@
 	(symbol
 		(lib_id "Device:R")
-		(at 68.58 80.01 0)
+		(at 68.58 78.74 0)
 		(mirror x)
 		(unit 1)
@@
 		(dnp no)
 		(property "Reference" "R11"
-			(at 72.39 78.74 0)
-			(show_name no)
-			(do_not_autoplace no)
-			(effects
-				(font
-					(size 1.27 1.27)
-				)
-			)
-		)
-		(property "Value" "100K"
-			(at 72.39 81.28 0)
+			(at 72.39 77.47 0)
+			(show_name no)
+			(do_not_autoplace no)
+			(effects
+				(font
+					(size 1.27 1.27)
+				)
+			)
+		)
+		(property "Value" "10K"
+			(at 72.39 80.01 0)
 			(show_name no)
 			(do_not_autoplace no)
@@
 		)
 		(property "Footprint" "Resistor_SMD:R_0805_2012Metric_Pad1.20x1.40mm_HandSolder"
-			(at 66.802 80.01 90)
+			(at 66.802 78.74 90)
 			(hide yes)
 			(show_name no)
@@
 		)
 		(property "Datasheet" ""
-			(at 68.58 80.01 0)
+			(at 68.58 78.74 0)
 			(hide yes)
 			(show_name no)
@@
 		)
 		(property "Description" "Resistor"
-			(at 68.58 80.01 0)
-			(hide yes)
-			(show_name no)
+			(at 68.58 78.74 0)
+			(hide yes)
+			(show_name no)

Commit message: PCB both ir board: ok add LM393D 3d model
Parts:
- R10: value 32R -> 50R
- R11: value 10K -> 100k
- R9: value 1K -> 1k
Changed lines of the file:
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@@
 			)
 		)
-		(property "Value" "10K"
+		(property "Value" "100k"
 			(at 72.39 80.01 0)
 			(show_name no)
@@
 			)
 		)
-		(property "Value" "32R"
+		(property "Value" "50R"
 			(at 68.58 62.23 90)
 			(show_name no)
@@
 			)
 		)
-		(property "Value" "1K"
+		(property "Value" "1k"
 			(at 62.23 74.93 90)
 			(show_name no)
