File: PCB/ChuniController/IRReceiver.kicad_sch (KiCad schematic)
At the start: 5 parts, among them Q3 Q_Photo_NPN, Q4 Q_Photo_NPN, U4 LM393D

Commit message: PCB + CAD
Parts:
- Q1: renamed from Q4; footprint (none) -> LED_THT:LED_D5.0mm
- Q2: renamed from Q3; footprint (none) -> LED_THT:LED_D5.0mm
- R3: renamed from R5; footprint (none) -> Resistor_SMD:R_0805_2012Metric_Pad1.20x1.40mm_HandSolder
- R4: footprint (none) -> Resistor_SMD:R_0805_2012Metric_Pad1.20x1.40mm_HandSolder
- renumbered U4 to U3
Changed lines of the file:
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@@
 		(dnp no)
 		(fields_autoplaced yes)
-		(property "Reference" "#PWR021"
+		(property "Reference" "#PWR013"
 			(at 152.4 62.23 0)
 			(hide yes)
@@
 			(project "ChuniController"
 				(path "/78a07370-9529-4114-be30-8ab9d3e7e0cd/4dd27aa0-f8f0-4f19-b021-a4827a7a836a/2ed5debb-a3d8-4999-8321-d2bf386ad2f4"
-					(reference "#PWR021")
+					(reference "#PWR013")
 					(unit 1)
 				)
 				(path "/78a07370-9529-4114-be30-8ab9d3e7e0cd/4dd27aa0-f8f0-4f19-b021-a4827a7a836a/43cddcc1-42a2-4b3a-8ca7-386440085070"
-					(reference "#PWR027")
+					(reference "#PWR025")
 					(unit 1)
 				)
 				(path "/78a07370-9529-4114-be30-8ab9d3e7e0cd/4dd27aa0-f8f0-4f19-b021-a4827a7a836a/b8778464-45a8-40a8-8839-569167ca584a"
-					(reference "#PWR029")
+					(reference "#PWR019")
 					(unit 1)
 				)
@@
 		(dnp no)
 		(fields_autoplaced yes)
-		(property "Reference" "#PWR022"
+		(property "Reference" "#PWR014"
 			(at 162.56 82.55 0)
 			(hide yes)
@@
 			(project "ChuniController"
 				(path "/78a07370-9529-4114-be30-8ab9d3e7e0cd/4dd27aa0-f8f0-4f19-b021-a4827a7a836a/2ed5debb-a3d8-4999-8321-d2bf386ad2f4"
-					(reference "#PWR022")
+					(reference "#PWR014")
 					(unit 1)
 				)
 				(path "/78a07370-9529-4114-be30-8ab9d3e7e0cd/4dd27aa0-f8f0-4f19-b021-a4827a7a836a/43cddcc1-42a2-4b3a-8ca7-386440085070"
-					(reference "#PWR028")
+					(reference "#PWR026")
 					(unit 1)
 				)
 				(path "/78a07370-9529-4114-be30-8ab9d3e7e0cd/4dd27aa0-f8f0-4f19-b021-a4827a7a836a/b8778464-45a8-40a8-8839-569167ca584a"
-					(reference "#PWR030")
+					(reference "#PWR020")
 					(unit 1)
 				)
@@
 			)
 		)
-		(property "Footprint" ""
+		(property "Footprint" "Resistor_SMD:R_0805_2012Metric_Pad1.20x1.40mm_HandSolder"
 			(at 41.402 97.79 90)
 			(hide yes)
@@
 				)
 				(path "/78a07370-9529-4114-be30-8ab9d3e7e0cd/4dd27aa0-f8f0-4f19-b021-a4827a7a836a/b8778464-45a8-40a8-8839-569167ca584a"
-					(reference "R9")
+					(reference "R6")
 					(unit 1)
 				)
@@
 		(dnp no)
 		(fields_autoplaced yes)
-		(property "Reference" "#PWR014"
+		(property "Reference" "#PWR011"
 			(at 43.18 81.28 0)
 			(hide yes)
@@
 			(project "ChuniController"
 				(path "/78a07370-9529-4114-be30-8ab9d3e7e0cd/4dd27aa0-f8f0-4f19-b021-a4827a7a836a/2ed5debb-a3d8-4999-8321-d2bf386ad2f4"
-					(reference "#PWR014")
+					(reference "#PWR011")
 					(unit 1)
 				)
 				(path "/78a07370-9529-4114-be30-8ab9d3e7e0cd/4dd27aa0-f8f0-4f19-b021-a4827a7a836a/43cddcc1-42a2-4b3a-8ca7-386440085070"
-					(reference "#PWR025")
+					(reference "#PWR023")
 					(unit 1)
 				)
 				(path "/78a07370-9529-4114-be30-8ab9d3e7e0cd/4dd27aa0-f8f0-4f19-b021-a4827a7a836a/b8778464-45a8-40a8-8839-569167ca584a"
-					(reference "#PWR019")
+					(reference "#PWR017")
 					(unit 1)
 				)
@@
 		(dnp no)
 		(fields_autoplaced yes)
-		(property "Reference" "#PWR016"
+		(property "Reference" "#PWR010"
 			(at 36.83 93.98 0)
 			(hide yes)
@@
 			(project "ChuniController"
 				(path "/78a07370-9529-4114-be30-8ab9d3e7e0cd/4dd27aa0-f8f0-4f19-b021-a4827a7a836a/2ed5debb-a3d8-4999-8321-d2bf386ad2f4"
+					(reference "#PWR010")
+					(unit 1)
+				)
+				(path "/78a07370-9529-4114-be30-8ab9d3e7e0cd/4dd27aa0-f8f0-4f19-b021-a4827a7a836a/43cddcc1-42a2-4b3a-8ca7-386440085070"
+					(reference "#PWR022")
+					(unit 1)
+				)
+				(path "/78a07370-9529-4114-be30-8ab9d3e7e0cd/4dd27aa0-f8f0-4f19-b021-a4827a7a836a/b8778464-45a8-40a8-8839-569167ca584a"
 					(reference "#PWR016")
-					(unit 1)
-				)
-				(path "/78a07370-9529-4114-be30-8ab9d3e7e0cd/4dd27aa0-f8f0-4f19-b021-a4827a7a836a/43cddcc1-42a2-4b3a-8ca7-386440085070"
-					(reference "#PWR024")
-					(unit 1)
-				)
-				(path "/78a07370-9529-4114-be30-8ab9d3e7e0cd/4dd27aa0-f8f0-4f19-b021-a4827a7a836a/b8778464-45a8-40a8-8839-569167ca584a"
-					(reference "#PWR018")
 					(unit 1)
 				)
@@
 		(dnp no)
 		(fields_autoplaced yes)
-		(property "Reference" "Q4"
+		(property "Reference" "Q1"
 			(at 37.3507 60.96 90)
 			(show_name no)
@@
 			)
 		)
-		(property "Footprint" ""
+		(property "Footprint" "LED_THT:LED_D5.0mm"
 			(at 35.56 64.77 0)
 			(hide yes)
@@
 			(project "ChuniController"
 				(path "/78a07370-9529-4114-be30-8ab9d3e7e0cd/4dd27aa0-f8f0-4f19-b021-a4827a7a836a/2ed5debb-a3d8-4999-8321-d2bf386ad2f4"
-					(reference "Q4")
+					(reference "Q1")
 					(unit 1)
 				)
 				(path "/78a07370-9529-4114-be30-8ab9d3e7e0cd/4dd27aa0-f8f0-4f19-b021-a4827a7a836a/43cddcc1-42a2-4b3a-8ca7-386440085070"
-					(reference "Q6")
+					(reference "Q5")
 					(unit 1)
 				)
 				(path "/78a07370-9529-4114-be30-8ab9d3e7e0cd/4dd27aa0-f8f0-4f19-b021-a4827a7a836a/b8778464-45a8-40a8-8839-569167ca584a"
-					(reference "Q5")
+					(reference "Q3")
 					(unit 1)
 				)
@@
 		(dnp no)
 		(fields_autoplaced yes)
-		(property "Reference" "R5"
+		(property "Reference" "R3"
 			(at 45.72 69.8499 0)
 			(show_name no)
@@
 			)
 		)
-		(property "Footprint" ""
+		(property "Footprint" "Resistor_SMD:R_0805_2012Metric_Pad1.20x1.40mm_HandSolder"
 			(at 41.402 71.12 90)
 			(hide yes)
@@
 			(project "ChuniController"
 				(path "/78a07370-9529-4114-be30-8ab9d3e7e0cd/4dd27aa0-f8f0-4f19-b021-a4827a7a836a/2ed5debb-a3d8-4999-8321-d2bf386ad2f4"
-					(reference "R5")
+					(reference "R3")
 					(unit 1)
 				)
@@
 				)
 				(path "/78a07370-9529-4114-be30-8ab9d3e7e0cd/4dd27aa0-f8f0-4f19-b021-a4827a7a836a/b8778464-45a8-40a8-8839-569167ca584a"
-					(reference "R6")
+					(reference "R5")
 					(unit 1)
 				)
@@
 		(dnp no)
 		(fields_autoplaced yes)
-		(property "Reference" "Q3"
+		(property "Reference" "Q2"
 			(at 37.3507 87.63 90)
 			(show_name no)
@@
 			)
 		)
-		(property "Footprint" ""
+		(property "Footprint" "LED_THT:LED_D5.0mm"
 			(at 35.56 91.44 0)
 			(hide yes)
@@
 			(project "ChuniController"
 				(path "/78a07370-9529-4114-be30-8ab9d3e7e0cd/4dd27aa0-f8f0-4f19-b021-a4827a7a836a/2ed5debb-a3d8-4999-8321-d2bf386ad2f4"
-					(reference "Q3")
+					(reference "Q2")
 					(unit 1)
 				)
 				(path "/78a07370-9529-4114-be30-8ab9d3e7e0cd/4dd27aa0-f8f0-4f19-b021-a4827a7a836a/43cddcc1-42a2-4b3a-8ca7-386440085070"
-					(reference "Q7")
+					(reference "Q6")
 					(unit 1)
 				)
 				(path "/78a07370-9529-4114-be30-8ab9d3e7e0cd/4dd27aa0-f8f0-4f19-b021-a4827a7a836a/b8778464-45a8-40a8-8839-569167ca584a"
-					(reference "Q8")
+					(reference "Q4")
 					(unit 1)
 				)
@@
 		(dnp no)
 		(fields_autoplaced yes)
-		(property "Reference" "U4"
+		(property "Reference" "U3"
 			(at 129.54 54.61 0)
 			(show_name no)
@@
 			(project "ChuniController"
 				(path "/78a07370-9529-4114-be30-8ab9d3e7e0cd/4dd27aa0-f8f0-4f19-b021-a4827a7a836a/2ed5debb-a3d8-4999-8321-d2bf386ad2f4"
-					(reference "U4")
+					(reference "U3")
 					(unit 1)
 				)
@@
 				)
 				(path "/78a07370-9529-4114-be30-8ab9d3e7e0cd/4dd27aa0-f8f0-4f19-b021-a4827a7a836a/b8778464-45a8-40a8-8839-569167ca584a"
-					(reference "U6")
+					(reference "U4")
 					(unit 1)
 				)
@@
 		(dnp no)
 		(fields_autoplaced yes)
-		(property "Reference" "#PWR013"
+		(property "Reference" "#PWR012"
 			(at 43.18 107.95 0)
 			(hide yes)
@@
 			(project "ChuniController"
 				(path "/78a07370-9529-4114-be30-8ab9d3e7e0cd/4dd27aa0-f8f0-4f19-b021-a4827a7a836a/2ed5debb-a3d8-4999-8321-d2bf386ad2f4"
-					(reference "#PWR013")
+					(reference "#PWR012")
 					(unit 1)
 				)
 				(path "/78a07370-9529-4114-be30-8ab9d3e7e0cd/4dd27aa0-f8f0-4f19-b021-a4827a7a836a/43cddcc1-42a2-4b3a-8ca7-386440085070"
-					(reference "#PWR026")
+					(reference "#PWR024")
 					(unit 1)
 				)
 				(path "/78a07370-9529-4114-be30-8ab9d3e7e0cd/4dd27aa0-f8f0-4f19-b021-a4827a7a836a/b8778464-45a8-40a8-8839-569167ca584a"
-					(reference "#PWR020")
+					(reference "#PWR018")
 					(unit 1)
 				)
@@
 		(dnp no)
 		(fields_autoplaced yes)
-		(property "Reference" "#PWR015"
+		(property "Reference" "#PWR09"
 			(at 36.83 67.31 0)
 			(hide yes)
@@
 			(project "ChuniController"
 				(path "/78a07370-9529-4114-be30-8ab9d3e7e0cd/4dd27aa0-f8f0-4f19-b021-a4827a7a836a/2ed5debb-a3d8-4999-8321-d2bf386ad2f4"
+					(reference "#PWR09")
+					(unit 1)
+				)
+				(path "/78a07370-9529-4114-be30-8ab9d3e7e0cd/4dd27aa0-f8f0-4f19-b021-a4827a7a836a/43cddcc1-42a2-4b3a-8ca7-386440085070"
+					(reference "#PWR021")
+					(unit 1)
+				)
+				(path "/78a07370-9529-4114-be30-8ab9d3e7e0cd/4dd27aa0-f8f0-4f19-b021-a4827a7a836a/b8778464-45a8-40a8-8839-569167ca584a"
 					(reference "#PWR015")
 					(unit 1)
 				)
-				(path "/78a07370-9529-4114-be30-8ab9d3e7e0cd/4dd27aa0-f8f0-4f19-b021-a4827a7a836a/43cddcc1-42a2-4b3a-8ca7-386440085070"
-					(reference "#PWR023")
-					(unit 1)
-				)
-				(path "/78a07370-9529-4114-be30-8ab9d3e7e0cd/4dd27aa0-f8f0-4f19-b021-a4827a7a836a/b8778464-45a8-40a8-8839-569167ca584a"
-					(reference "#PWR017")
-					(unit 1)
-				)

Commit message: PCB Add pullup 10kR in LM393D reduce AO3400 pulldown to 10kR
Parts:
- added R27, R30: 10k, symbol Device:R
Connections:
- net +3V3: now also R27.1, R30.1
- net OUT_1: now also R27.2
- net OUT_2: now also R30.2

Commit message: PCB both ir board: ok add LM393D 3d model
Parts:
- R27, R30: footprint (none) -> Resistor_SMD:R_0805_2012Metric_Pad1.20x1.40mm_HandSolder
Other:
- moved on the sheet: R3
Changed lines of the file:
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@@
 	)
 	(junction
-		(at 43.18 67.31)
+		(at 45.72 67.31)
 		(diameter 0)
 		(color 0 0 0 0)
@@
 	(wire
 		(pts
-			(xy 43.18 67.31) (xy 111.76 67.31)
+			(xy 43.18 67.31) (xy 45.72 67.31)
 		)
 		(stroke
@@
 		(pts
 			(xy 153.67 64.77) (xy 153.67 67.31)
+		)
+		(stroke
+			(width 0)
+			(type default)
+		)
+	)
+	(wire
+		(pts
+			(xy 45.72 67.31) (xy 111.76 67.31)
 		)
 		(stroke
@@
 	(symbol
 		(lib_id "power:GND")
-		(at 43.18 74.93 0)
+		(at 45.72 74.93 0)
 		(unit 1)
 		(body_style 1)
@@
 		(fields_autoplaced yes)
 		(property "Reference" "#PWR011"
-			(at 43.18 81.28 0)
+			(at 45.72 81.28 0)
 			(hide yes)
 			(show_name no)
@@
 		)
 		(property "Value" "GND"
-			(at 43.18 80.01 0)
+			(at 45.72 80.01 0)
 			(show_name no)
 			(do_not_autoplace no)
@@
 		)
 		(property "Footprint" ""
-			(at 43.18 74.93 0)
+			(at 45.72 74.93 0)
 			(hide yes)
 			(show_name no)
@@
 		)
 		(property "Datasheet" ""
-			(at 43.18 74.93 0)
+			(at 45.72 74.93 0)
 			(hide yes)
 			(show_name no)
@@
 		)
 		(property "Description" "Power symbol creates a global label with name \"GND\" , ground"
-			(at 43.18 74.93 0)
+			(at 45.72 74.93 0)
 			(hide yes)
 			(show_name no)
@@
 			)
 		)
-		(property "Footprint" ""
+		(property "Footprint" "Resistor_SMD:R_0805_2012Metric_Pad1.20x1.40mm_HandSolder"
 			(at 151.892 60.96 90)
 			(hide yes)
@@
 	(symbol
 		(lib_id "Device:R")
-		(at 43.18 71.12 0)
+		(at 45.72 71.12 0)
 		(unit 1)
 		(body_style 1)
@@
 		(fields_autoplaced yes)
 		(property "Reference" "R3"
-			(at 45.72 69.8499 0)
+			(at 48.26 69.8499 0)
 			(show_name no)
 			(do_not_autoplace no)
@@
 		)
 		(property "Value" "30k"
-			(at 45.72 72.3899 0)
+			(at 48.26 72.3899 0)
 			(show_name no)
 			(do_not_autoplace no)
@@
 		)
 		(property "Footprint" "Resistor_SMD:R_0805_2012Metric_Pad1.20x1.40mm_HandSolder"
-			(at 41.402 71.12 90)
+			(at 43.942 71.12 90)
 			(hide yes)
 			(show_name no)
@@
 		)
 		(property "Datasheet" ""
-			(at 43.18 71.12 0)
+			(at 45.72 71.12 0)
 			(hide yes)
 			(show_name no)
@@
 		)
 		(property "Description" "Resistor"
-			(at 43.18 71.12 0)
+			(at 45.72 71.12 0)
 			(hide yes)
 			(show_name no)
@@
 			)
 		)
-		(property "Footprint" ""
+		(property "Footprint" "Resistor_SMD:R_0805_2012Metric_Pad1.20x1.40mm_HandSolder"
 			(at 155.702 60.96 90)
 			(hide yes)
